Commit message: correct params

File: src/turn_on_diode_robot/urdf/mini_mec_robot.urdf (robot description, URDF)
Before this commit: robot diode_robot, 5 links, 4 joints
Joints:
- joint left_front_joint: origin xyz=0.085 0.0975 0.0375 rpy=1.57 0 0 -> xyz=0.2 0.2 0.09 rpy=0 0 0
- joint left_wheel_joint: origin xyz=-0.085 0.0975 0.0375 rpy=1.57 0 0 -> xyz=-0.2 0.2 0.09 rpy=0 0 0
- joint right_front_joint: origin xyz=0.085 -0.0975 0.0375 rpy=1.57 0 0 -> xyz=0.2 -0.2 0.09 rpy=0 0 0
- joint right_wheel_joint: origin xyz=-0.085 -0.0975 0.0375 rpy=1.57 0 0 -> xyz=-0.2 -0.2 0.09 rpy=0 0 0

Commit message: mid360 will ok

File: src/turn_on_diode_robot/urdf/mini_mec_robot.urdf (robot description, URDF)
Before this commit: robot diode_robot, 5 links, 4 joints
Joints:
- joint left_front_joint: origin xyz=0.2 0.2 0.09 rpy=0 0 0 -> xyz=0.085 0.0975 0.0375 rpy=1.57 0 0
- joint left_wheel_joint: origin xyz=-0.2 0.2 0.09 rpy=0 0 0 -> xyz=-0.085 0.0975 0.0375 rpy=1.57 0 0
- joint right_front_joint: origin xyz=0.2 -0.2 0.09 rpy=0 0 0 -> xyz=0.085 -0.0975 0.0375 rpy=1.57 0 0
- joint right_wheel_joint: origin xyz=-0.2 -0.2 0.09 rpy=0 0 0 -> xyz=-0.085 -0.0975 0.0375 rpy=1.57 0 0
